Commit message: Replace original names with new package name .

File: navigation_config/gazebo_test_config/description/urdf/livox_mid360.urdf.xacro (robot description, xacro)
@@ -34,5 +34,5 @@
                 <origin xyz="0 0 0" rpy="0 0 0"/>
                 <geometry>
-                    <mesh filename="package://navigation_config/description/meshes/lidar/livox_mid360.stl" scale="1 1 1"/>
+                    <mesh filename="package://gazebo_test_config/description/meshes/lidar/livox_mid360.stl" scale="1 1 1"/>
                 </geometry>
             </visual>

File: navigation_config/gazebo_test_config/description/urdf/ranger_livox.xacro (robot description, xacro)
@@ -2,6 +2,6 @@
 <robot xmlns:xacro="http://ros.org/wiki/xacro" name="ranger_livox">
     <xacro:arg name="use_simulation" default="true"/>
-    <xacro:include filename="$(find navigation_config)/description/urdf/livox_mid360.urdf.xacro"/>
-    <xacro:include filename="$(find navigation_config)/description/urdf/ranger_mini_gazebo.xacro"/>
+    <xacro:include filename="$(find gazebo_test_config)/description/urdf/livox_mid360.urdf.xacro"/>
+    <xacro:include filename="$(find gazebo_test_config)/description/urdf/ranger_mini_gazebo.xacro"/>
     <xacro:livox_mid360 connected_to="base_link" simulation="true" lidar_name="livox_lidar" imu_name="livox_imu"
                         xyz="0.0 0.0 0.055" rpy="0.0 0.0 0.0"/>

File: navigation_config/gazebo_test_config/description/urdf/ranger_mini_gazebo.xacro (robot description, xacro)
@@ -12,5 +12,5 @@
 <!--            <origin xyz="0 0 0" rpy="1.57 0 3.14 " />-->
 <!--            <geometry>-->
-<!--                <mesh filename="package://navigation_config/description/meshes/ranger_mini_v2/ranger_base/ranger_base.dae" />-->
+<!--                <mesh filename="package://gazebo_test_config/description/meshes/ranger_mini_v2/ranger_base/ranger_base.dae" />-->
 <!--            </geometry>-->
             <origin xyz="0 0 -0.1" rpy="0 0 0" />
@@ -35,5 +35,5 @@
 <!--            <origin xyz="-0.23 -0.194 0.1" rpy="1.57 0 3.14 " />-->
 <!--            <geometry>-->
-<!--                    <mesh filename="package://navigation_config/description/meshes/ranger_mini_v2/fl.dae" />-->
+<!--                    <mesh filename="package://gazebo_test_config/description/meshes/ranger_mini_v2/fl.dae" />-->
 <!--            </geometry>-->
             <origin xyz="0 0 0" rpy="0 0 0" />
@@ -109,5 +109,5 @@
 <!--            <origin xyz="-0.23 0.194 0.1" rpy="1.57 0 3.14 " />-->
 <!--            <geometry>-->
-<!--                <mesh filename="package://navigation_config/description/meshes/ranger_mini_v2/fr.dae" />-->
+<!--                <mesh filename="package://gazebo_test_config/description/meshes/ranger_mini_v2/fr.dae" />-->
 <!--            </geometry>-->
         </visual>
@@ -173,5 +173,5 @@
 <!--            <origin xyz="-0.23 -0.194 0.1" rpy="1.57 0 3.14 " />-->
 <!--            <geometry>-->
-<!--                    <mesh filename="package://navigation_config/description/meshes/ranger_mini_v2/fl.dae" />-->
+<!--                    <mesh filename="package://gazebo_test_config/description/meshes/ranger_mini_v2/fl.dae" />-->
 <!--            </geometry>-->
         </visual>
@@ -237,5 +237,5 @@
 <!--            <origin xyz="-0.23 0.194 0.1" rpy="1.57 0 3.14 " />-->
 <!--            <geometry>-->
-<!--                    <mesh filename="package://navigation_config/description/meshes/ranger_mini_v2/fr.dae" />-->
+<!--                    <mesh filename="package://gazebo_test_config/description/meshes/ranger_mini_v2/fr.dae" />-->
 <!--            </geometry>-->
         </visual>
